Commit message: Repo Update

File: husky_ur3_gazebo/urdf/accessories/d435_camera_g.urdf.xacro (robot description, xacro)
@@ -139,5 +139,5 @@
             <visualize>true</visualize>
             <camera>
-                <horizontal_fov>${60*M_PI/180.0}</horizontal_fov>
+                <horizontal_fov>${86*M_PI/180.0}</horizontal_fov>
                 <image>
                     <width>640</width>
@@ -148,5 +148,5 @@
                 </depth_camera>
                 <clip>
-                    <near>0.11</near>
+                    <near>0.01</near>
                     <far>10</far>
                 </clip>

File: husky_ur3_gazebo/urdf/accessories/d435_camera_h.urdf.xacro (robot description, xacro)
@@ -139,5 +139,5 @@
             <visualize>true</visualize>
             <camera>
-                <horizontal_fov>${60*M_PI/180.0}</horizontal_fov>
+                <horizontal_fov>${86*M_PI/180.0}</horizontal_fov>
                 <image>
                     <width>640</width>
@@ -148,5 +148,5 @@
                 </depth_camera>
                 <clip>
-                    <near>0.11</near>
+                    <near>0.01</near>
                     <far>10</far>
                 </clip>

File: husky_ur3_gazebo/urdf/decorations.urdf.xacro (robot description, xacro)
@@ -207,5 +207,5 @@
     </joint>-->
     <xacro:h_sensor_d435 parent="top_plate_link">
-        <origin xyz="0.4 0.0 0.06" rpy="0 0 0"/>
+        <origin xyz="0.4 0.0 0.00" rpy="0 0 0"/>
     </xacro:h_sensor_d435>
   </xacro:macro>

File: husky_ur3_gazebo/urdf/husky_ur3_gripper.urdf.xacro (robot description, xacro)
@@ -24,8 +24,19 @@
   <xacro:arg name="laser_xyz" default="$(optenv HUSKY_LMS1XX_XYZ 0.3206 0.0 -0.000635)" />
   <xacro:arg name="laser_rpy" default="$(optenv HUSKY_LMS1XX_RPY 0.0 0 0)" />
+  <!-- camera_h: decorations.urdf.xacro -->
+  <!-- camera_g: ur3_robot_gripper.urdf.xacro -->
+  <!--
+  <xacro:arg name="camera_h_enabled" default="true" />
+  <xacro:arg name="camera_g_enabled" default="true" />
+  <xacro:arg name="camera_h_xyz" default="$(optenv HUSKY_KINECT_XYZ 0.33 0 0.01)" />
+  <xacro:arg name="camera_h_rpy" default="$(optenv HUSKY_KINECT_RPY 0 -0.314 0)" />
+  <xacro:arg name="camera_g_xyz" default="$(optenv HUSKY_KINECT_XYZ 0 0 0.04)" />
+  <xacro:arg name="camera_g_rpy" default="$(optenv HUSKY_KINECT_RPY 0 0 0)" />
+  -->
   <xacro:property name="husky_front_bumper_extend" value="$(optenv HUSKY_FRONT_BUMPER_EXTEND 0)" />
   <xacro:property name="husky_rear_bumper_extend" value="$(optenv HUSKY_REAR_BUMPER_EXTEND 0)" />
   <xacro:arg name="robot_namespace" default="/husky" />
   <xacro:arg name="urdf_extras" default="empty.urdf" />
+  <xacro:arg name="transmission_hw_interface" default="false"/>
   <!-- Included URDF/XACRO Files -->
   <xacro:include filename="$(find husky_ur3_gazebo)/urdf/decorations.urdf.xacro" />
@@ -33,7 +44,12 @@
   <xacro:include filename="$(find husky_ur3_gazebo)/urdf/accessories/sensor_arch.urdf.xacro"/>
   <xacro:include filename="$(find husky_ur3_gazebo)/urdf/accessories/sick_tim571.urdf.xacro"/>
-  <xacro:include filename="$(find husky_ur3_gazebo)/urdf/ur3_robot_gripper.urdf.xacro"/>
-  <xacro:include filename="$(find husky_ur3_gazebo)/urdf/accessories/d435_camera_h.urdf.xacro"/>-
-  <xacro:include filename="$(find husky_ur3_gazebo)/urdf/accessories/d435_camera_g.urdf.xacro"/>-
+  <xacro:if value="$(arg transmission_hw_interface)">
+    <xacro:include filename="$(find husky_ur3_gazebo)/urdf/ur3_robot_gripper_effort.urdf.xacro"/>
+  </xacro:if>
+  <xacro:unless value="$(arg transmission_hw_interface)">
+    <xacro:include filename="$(find husky_ur3_gazebo)/urdf/ur3_robot_gripper.urdf.xacro"/>
+  </xacro:unless>
+  <xacro:include filename="$(find husky_ur3_gazebo)/urdf/accessories/d435_camera_h.urdf.xacro"/>
+  <xacro:include filename="$(find husky_ur3_gazebo)/urdf/accessories/d435_camera_g.urdf.xacro"/>
   <!--xacro:include filename="$(find husky_ur3_gazebo)/urdf/ur3_robot.urdf.xacro"/-->
   <xacro:property name="M_PI" value="3.14159"/>
@@ -153,4 +169,15 @@
    	<origin xyz="$(arg laser_xyz)" rpy="$(arg laser_rpy)"/>
   </xacro:sensor_sick_tim571>
+<!--  <xacro:if value="$(arg camera_h_enabled)">
+    <xacro:h_sensor_d435 parent="top_plate_link">
+      <origin xyz="$(arg camera_h_xyz)" rpy="$(arg camera_h_rpy)"/>
+    </xacro:h_sensor_d435>
+  </xacro:if>
+  <xacro:if value="$(arg camera_g_enabled)">
+    <xacro:g_sensor_d435 parent="ee_link">
+      <origin xyz="$(arg camera_g_xyz)" rpy="$(arg camera_g_rpy)"/>
+    </xacro:g_sensor_d435>
+  </xacro:if>
+-->
  <joint name="control_box_ur3_joint" type="fixed">
       <origin xyz="-0.095 0 0.233" rpy="${M_PI/2} 0 0" />
@@ -219,3 +246,20 @@
   <!-- Optional custom includes. -->
   <xacro:include filename="$(arg urdf_extras)" />
+  <gazebo>
+    <plugin name="gazebo_grasp_fix" filename="libgazebo_grasp_fix.so">
+        <arm>
+          <arm_name>ur3_robot</arm_name>
+          <palm_link> wrist_3_link  </palm_link>
+          <gripper_link> rh_p12_rn_r2 </gripper_link>
+          <gripper_link> rh_p12_rn_l2 </gripper_link>
+        </arm>
+        <forces_angle_tolerance>100</forces_angle_tolerance>
+        <update_rate>4</update_rate>
+        <grip_count_threshold>4</grip_count_threshold>
+        <max_grip_count>8</max_grip_count>
+        <release_tolerance>0.005</release_tolerance>
+        <disable_collisions_on_attach>false</disable_collisions_on_attach>
+        <contact_topic>__default_topic__</contact_topic>
+    </plugin>
+  </gazebo>
 </robot>

File: husky_ur3_gazebo/urdf/ur3.urdf.xacro (robot description, xacro)
@@ -22,5 +22,5 @@
     wrist_2_lower_limit:=${-pi}    wrist_2_upper_limit:=${pi}
     wrist_3_lower_limit:=${-pi}    wrist_3_upper_limit:=${pi}
-    transmission_hw_interface:=hardware_interface/PositionJointInterface
+    transmission_hw_interface
     safety_limits:=false safety_pos_margin:=0.15
     safety_k_position:=20">

File: husky_ur3_gazebo/urdf/ur3_robot_gripper.urdf.xacro (robot description, xacro)
@@ -2,5 +2,5 @@
 <robot xmlns:xacro="http://wiki.ros.org/xacro"
        name="ur3" >
-  <xacro:arg name="transmission_hw_interface" default="hardware_interface/PositionJointInterface"/>
+  <xacro:arg name="transmission_hw_interface" default="hardware_interface/EffortJointInterface"/>
   <!-- common stuff -->
   <!--xacro:include filename="$(find ur_description)/urdf/common.gazebo.xacro" /-->
@@ -17,5 +17,5 @@
     wrist_2_lower_limit="${-pi}" wrist_2_upper_limit="${pi}"
     wrist_3_lower_limit="${-pi}" wrist_3_upper_limit="${pi}"
-    transmission_hw_interface="$(arg transmission_hw_interface)"
+    transmission_hw_interface="hardware_interface/PositionJointInterface"
   />
   <joint name="husky_ur3_joint" type="fixed">
