Commit message: Fix lidar plugin length

File: husky_ur3_gazebo/urdf/accessories/sick_tim571.urdf.xacro (robot description, xacro)
@@ -1,70 +1,71 @@
 <?xml version="1.0"?>
 <robot xmlns:xacro="http://www.ros.org/wiki/xacro">
-  <xacro:macro name="sensor_sick_tim571" params="prefix parent prefix_topic:='front_laser' *origin min_angle:=-1.57619449019 max_angle:=1.57619449019">
+  <xacro:macro name="sensor_sick_tim571"
+    params="prefix parent prefix_topic:='front_laser' *origin min_angle:=-1.57619449019 max_angle:=1.57619449019">
     <joint name="${prefix}_base_joint" type="fixed">
       <xacro:insert_block name="origin" />
-      <parent link="${parent}"/>
-      <child link="${prefix}_base_link"/>
+      <parent link="${parent}" />
+      <child link="${prefix}_base_link" />
     </joint>
     <link name="${prefix}_base_link">
       <collision>
-        <origin xyz="0 0 0" rpy="3.1415926 0 0"/>
+        <origin xyz="0 0 0" rpy="3.1415926 0 0" />
         <geometry>
-         <mesh filename="package://husky_ur3_gazebo/meshes/sick_tim/sick_tim571.dae"/>
+          <mesh filename="package://husky_ur3_gazebo/meshes/sick_tim/sick_tim571.dae" />
         </geometry>
       </collision>
       <visual>
-        <origin xyz="0 0 0" rpy="3.1415926 0 0"/>
+        <origin xyz="0 0 0" rpy="3.1415926 0 0" />
         <geometry>
-            <mesh filename="package://husky_ur3_gazebo/meshes/sick_tim/sick_tim571.dae"/>
+          <mesh filename="package://husky_ur3_gazebo/meshes/sick_tim/sick_tim571.dae" />
         </geometry>
       </visual>
       <inertial>
         <mass value="1e-5" />
-        <origin xyz="0 0 0" rpy="3.1415926 0 0"/>
+        <origin xyz="0 0 0" rpy="3.1415926 0 0" />
         <inertia ixx="1e-6" ixy="0" ixz="0" iyy="1e-6" iyz="0" izz="1e-6" />
       </inertial>
     </link>
     <joint name="${prefix}_joint" type="fixed">
-      <origin xyz="0 0 -0.06246" rpy="0 0 0"/>
-      <parent link="${prefix}_base_link"/>
-      <child link="${prefix}_link"/>
+      <origin xyz="0 0 -0.06246" rpy="0 0 0" />
+      <parent link="${prefix}_base_link" />
+      <child link="${prefix}_link" />
     </joint>
     <link name="${prefix}_link">
     </link>
-    <xacro:sensor_sick_tim571_gazebo/>
+    <xacro:sensor_sick_tim571_gazebo />
   </xacro:macro>
   <xacro:macro name="sensor_sick_tim571_gazebo">
-	<gazebo reference="${prefix}_link">
-			<sensor type="ray" name="${prefix}_sensor">
-				<pose>0 0 0 0 0 0</pose>
-				<visualize>false</visualize>
-				<update_rate>15</update_rate>
-				<ray>
-					<scan>
-						<horizontal>
-							<samples>716</samples>
-							<resolution>1</resolution>
-							<min_angle>${min_angle}</min_angle>
-							<max_angle>${max_angle}</max_angle>
-						</horizontal>
-					</scan>
-					<range>
-						<min>0.05</min>
-						<max>25.0</max>
-						<resolution>0.00575</resolution>
-					</range>
-					<noise>
-						<type>gaussian</type>
-						<mean>0.0</mean>
-						<stddev>0.01</stddev>
-					</noise>
-				</ray>
-				<plugin name="${prefix}_controller" filename="libgazebo_ros_laser.so">
-					<topicName>/scan</topicName>
-					<frameName>/${prefix}_link</frameName>
-				</plugin>
-			</sensor>
-	</gazebo>
+    <gazebo reference="${prefix}_link">
+      <sensor type="ray" name="${prefix}_sensor">
+        <pose>0 0 0 0 0 0</pose>
+        <visualize>false</visualize>
+        <update_rate>15</update_rate>
+        <ray>
+          <scan>
+            <horizontal>
+              <samples>609</samples>
+              <resolution>1</resolution>
+              <min_angle>${min_angle}</min_angle>
+              <max_angle>${max_angle}</max_angle>
+            </horizontal>
+          </scan>
+          <range>
+            <min>0.05</min>
+            <max>25.0</max>
+            <resolution>0.00575</resolution>
+          </range>
+          <noise>
+            <type>gaussian</type>
+            <mean>0.0</mean>
+            <stddev>0.01</stddev>
+          </noise>
+        </ray>
+        <plugin name="${prefix}_controller" filename="libgazebo_ros_laser.so">
+          <topicName>/scan</topicName>
+          <frameName>/${prefix}_link</frameName>
+        </plugin>
+      </sensor>
+    </gazebo>
   </xacro:macro>
 </robot>
