Commit message: Add collision sensor

File: husky_ur3_gazebo/urdf/decorations.urdf.xacro (robot description, xacro)
@@ -5,24 +5,36 @@
 \authors   Paul Bovbel <pbovbel@clearpathrobotics.com>, Devon Ash <dash@clearpathrobotics.com>
 \copyright Copyright (c) 2015, Clearpath Robotics, Inc., All rights reserved.
-Redistribution and use in source and binary forms, with or without modification, are permitted provided that
+Redistribution and use in source and binary forms, with or without modification, are permitted
+provided that
 the following conditions are met:
- * Redistributions of source code must retain the above copyright notice, this list of conditions and the
+ * Redistributions of source code must retain the above copyright notice, this list of conditions
+and the
    following disclaimer.
- * Redistributions in binary form must reproduce the above copyright notice, this list of conditions and the
+ * Redistributions in binary form must reproduce the above copyright notice, this list of conditions
+and the
    following disclaimer in the documentation and/or other materials provided with the distribution.
- * Neither the name of Clearpath Robotics nor the names of its contributors may be used to endorse or promote
+ * Neither the name of Clearpath Robotics nor the names of its contributors may be used to endorse
+or promote
    products derived from this software without specific prior written permission.
-THIS SOFTWARE IS PROVIDED BY THE COPYRIGHT HOLDERS AND CONTRIBUTORS "AS IS" AND ANY EXPRESS OR IMPLIED WAR-
-RANTIES, INCLUDING, BUT NOT LIMITED TO, THE IMPLIED WARRANTIES OF MERCHANTABILITY AND FITNESS FOR A PARTICULAR
-PURPOSE ARE DISCLAIMED. IN NO EVENT SHALL THE COPYRIGHT HOLDER OR CONTRIBUTORS BE LIABLE FOR ANY DIRECT, IN-
-DIRECT, INCIDENTAL, SPECIAL, EXEMPLARY, OR CONSEQUENTIAL DAMAGES (INCLUDING, BUT NOT LIMITED TO, PROCUREMENT
-OF SUBSTITUTE GOODS OR SERVICES; LOSS OF USE, DATA, OR PROFITS; OR BUSINESS INTERRUPTION) HOWEVER CAUSED AND
-ON ANY THEORY OF LIABILITY, WHETHER IN CONTRACT, STRICT LIABILITY, OR TORT (INCLUDING NEGLIGENCE OR OTHERWISE)
-ARISING IN ANY WAY OUT OF THE USE OF THIS SOFTWARE, EVEN IF ADVISED OF THE POSSIBILITY OF SUCH DAMAGE.
+THIS SOFTWARE IS PROVIDED BY THE COPYRIGHT HOLDERS AND CONTRIBUTORS "AS IS" AND ANY EXPRESS OR
+IMPLIED WAR-
+RANTIES, INCLUDING, BUT NOT LIMITED TO, THE IMPLIED WARRANTIES OF MERCHANTABILITY AND FITNESS FOR A
+PARTICULAR
+PURPOSE ARE DISCLAIMED. IN NO EVENT SHALL THE COPYRIGHT HOLDER OR CONTRIBUTORS BE LIABLE FOR ANY
+DIRECT, IN-
+DIRECT, INCIDENTAL, SPECIAL, EXEMPLARY, OR CONSEQUENTIAL DAMAGES (INCLUDING, BUT NOT LIMITED TO,
+PROCUREMENT
+OF SUBSTITUTE GOODS OR SERVICES; LOSS OF USE, DATA, OR PROFITS; OR BUSINESS INTERRUPTION) HOWEVER
+CAUSED AND
+ON ANY THEORY OF LIABILITY, WHETHER IN CONTRACT, STRICT LIABILITY, OR TORT (INCLUDING NEGLIGENCE OR
+OTHERWISE)
+ARISING IN ANY WAY OUT OF THE USE OF THIS SOFTWARE, EVEN IF ADVISED OF THE POSSIBILITY OF SUCH
+DAMAGE.
 -->
 <robot name="husky_decorations" xmlns:xacro="http://ros.org/wiki/xacro">
   <xacro:macro name="husky_decorate">
-    <xacro:property name="husky_front_bumper_extend" value="$(optenv HUSKY_FRONT_BUMPER_EXTEND 0)" />
-    <xacro:property name="husky_rear_bumper_extend" value="$(optenv HUSKY_REAR_BUMPER_EXTEND 0)" />
+    <xacro:property name="husky_front_bumper_extend"
+      value="$(optenv HUSKY_FRONT_BUMPER_EXTEND 0.01)" />
+    <xacro:property name="husky_rear_bumper_extend" value="$(optenv HUSKY_REAR_BUMPER_EXTEND 0.01)" />
     <!-- Spawn Husky chassis -->
     <link name="top_chassis_link">
@@ -62,4 +74,9 @@
         </geometry>
       </visual>
+      <collision name="front_bumper_collision">
+        <geometry>
+          <mesh filename="package://husky_ur3_gazebo/meshes/bumper.dae" />
+        </geometry>
+      </collision>
     </link>
     <!-- Attach front bumper -->
@@ -71,9 +88,9 @@
     <xacro:if value="${husky_front_bumper_extend}">
       <link name="front_bumper_extension_link">
-          <visual>
-              <geometry>
-                  <mesh filename="package://husky_ur3_gazebo/meshes/bumper_extension.dae" />
-              </geometry>
-          </visual>
+        <visual>
+          <geometry>
+            <mesh filename="package://husky_ur3_gazebo/meshes/bumper_extension.dae" />
+          </geometry>
+        </visual>
       </link>
       <joint name="front_bumper_extension" type="fixed">
@@ -90,4 +107,9 @@
         </geometry>
       </visual>
+      <collision name="rear_bumper_collision">
+        <geometry>
+          <mesh filename="package://husky_ur3_gazebo/meshes/bumper.dae" />
+        </geometry>
+      </collision>
     </link>
     <!-- Attach rear bumper -->
@@ -99,9 +121,9 @@
     <xacro:if value="${husky_rear_bumper_extend}">
       <link name="rear_bumper_extension_link">
-          <visual>
-              <geometry>
-                  <mesh filename="package://husky_ur3_gazebo/meshes/bumper_extension.dae" />
-              </geometry>
-          </visual>
+        <visual>
+          <geometry>
+            <mesh filename="package://husky_ur3_gazebo/meshes/bumper_extension.dae" />
+          </geometry>
+        </visual>
       </link>
       <joint name="rear_bumper_extension" type="fixed">
@@ -122,5 +144,5 @@
           </visual>
           <collision>
-            <origin xyz="0 0 0" rpy="0 0 0"/>
+            <origin xyz="0 0 0" rpy="0 0 0" />
             <geometry>
               <mesh filename="package://husky_ur3_gazebo/meshes/large_top_plate_collision.stl" />
@@ -131,18 +153,18 @@
         <joint name="top_plate_joint" type="fixed">
           <parent link="base_link" />
-          <child link="top_plate_link"/>
-          <origin xyz="0.0812 0 0.225" rpy="0 0 0"/>
+          <child link="top_plate_link" />
+          <origin xyz="0.0812 0 0.225" rpy="0 0 0" />
         </joint>
         <!-- Top plate front link -->
         <joint name="top_plate_front_joint" type="fixed">
           <parent link="top_plate_link" />
-          <child link="top_plate_front_link"/>
-          <origin xyz="0.4125 0 0.00672" rpy="0 0 0"/>
+          <child link="top_plate_front_link" />
+          <origin xyz="0.4125 0 0.00672" rpy="0 0 0" />
         </joint>
         <!-- Top plate rear link-->
         <joint name="top_plate_rear_joint" type="fixed">
           <parent link="top_plate_link" />
-          <child link="top_plate_rear_link"/>
-          <origin xyz="-0.4125 0 0.00672" rpy="0 0 0"/>
+          <child link="top_plate_rear_link" />
+          <origin xyz="-0.4125 0 0.00672" rpy="0 0 0" />
         </joint>
       </xacro:if>
@@ -156,5 +178,5 @@
           </visual>
           <collision>
-            <origin xyz="0 0 0" rpy="0 0 0"/>
+            <origin xyz="0 0 0" rpy="0 0 0" />
             <geometry>
               <mesh filename="package://husky_ur3_gazebo/meshes/top_plate.stl" />
@@ -165,25 +187,27 @@
         <joint name="top_plate_joint" type="fixed">
           <parent link="base_link" />
-          <child link="top_plate_link"/>
-          <origin xyz="0.0812 0 0.245" rpy="0 0 0"/>
+          <child link="top_plate_link" />
+          <origin xyz="0.0812 0 0.245" rpy="0 0 0" />
         </joint>
         <!-- Top plate front link -->
         <joint name="top_plate_front_joint" type="fixed">
           <parent link="top_plate_link" />
-          <child link="top_plate_front_link"/>
-          <origin xyz="0.36367 0 0.00639" rpy="0 0 0"/>
+          <child link="top_plate_front_link" />
+          <origin xyz="0.36367 0 0.00639" rpy="0 0 0" />
         </joint>
         <!-- Top plate rear link-->
         <joint name="top_plate_rear_joint" type="fixed">
           <parent link="top_plate_link" />
-          <child link="top_plate_rear_link"/>
-          <origin xyz="-0.36633 0 0.00639" rpy="0 0 0"/>
+          <child link="top_plate_rear_link" />
+          <origin xyz="-0.36633 0 0.00639" rpy="0 0 0" />
         </joint>
       </xacro:unless>
-      <link name="top_plate_front_link"/>
-      <link name="top_plate_rear_link"/>
-    </xacro:if>
-    <!--D435 mount frame -->
-    <!--<link name="mount_link">
+      <link name="top_plate_front_link" />
+      <link name="top_plate_rear_link" />
+    </xacro:if>
+    <!--D435
+    mount frame -->
+    <!--<link
+    name="mount_link">
         <visual>
             <geometry>
@@ -207,5 +231,5 @@
     </joint>-->
     <xacro:h_sensor_d435 parent="top_plate_link">
-        <origin xyz="0.4 0.0 0.00" rpy="0 0 0"/>
+      <origin xyz="0.4 0.0 0.06" rpy="0 0 0" />
     </xacro:h_sensor_d435>
   </xacro:macro>
