Commit message: Add collision sensor

File: husky_ur3_gazebo/urdf/husky_ur3_gripper.urdf.xacro (robot description, xacro)
@@ -5,19 +5,30 @@
 \authors   Paul Bovbel <pbovbel@clearpathrobotics.com>, Devon Ash <dash@clearpathrobotics.com>
 \copyright Copyright (c) 2015, Clearpath Robotics, Inc., All rights reserved.
-Redistribution and use in source and binary forms, with or without modification, are permitted provided that
+Redistribution and use in source and binary forms, with or without modification, are permitted
+provided that
 the following conditions are met:
- * Redistributions of source code must retain the above copyright notice, this list of conditions and the
+ * Redistributions of source code must retain the above copyright notice, this list of conditions
+and the
    following disclaimer.
- * Redistributions in binary form must reproduce the above copyright notice, this list of conditions and the
+ * Redistributions in binary form must reproduce the above copyright notice, this list of conditions
+and the
    following disclaimer in the documentation and/or other materials provided with the distribution.
- * Neither the name of Clearpath Robotics nor the names of its contributors may be used to endorse or promote
+ * Neither the name of Clearpath Robotics nor the names of its contributors may be used to endorse
+or promote
    products derived from this software without specific prior written permission.
-THIS SOFTWARE IS PROVIDED BY THE COPYRIGHT HOLDERS AND CONTRIBUTORS "AS IS" AND ANY EXPRESS OR IMPLIED WAR-
-RANTIES, INCLUDING, BUT NOT LIMITED TO, THE IMPLIED WARRANTIES OF MERCHANTABILITY AND FITNESS FOR A PARTICULAR
-PURPOSE ARE DISCLAIMED. IN NO EVENT SHALL THE COPYRIGHT HOLDER OR CONTRIBUTORS BE LIABLE FOR ANY DIRECT, IN-
-DIRECT, INCIDENTAL, SPECIAL, EXEMPLARY, OR CONSEQUENTIAL DAMAGES (INCLUDING, BUT NOT LIMITED TO, PROCUREMENT
-OF SUBSTITUTE GOODS OR SERVICES; LOSS OF USE, DATA, OR PROFITS; OR BUSINESS INTERRUPTION) HOWEVER CAUSED AND
-ON ANY THEORY OF LIABILITY, WHETHER IN CONTRACT, STRICT LIABILITY, OR TORT (INCLUDING NEGLIGENCE OR OTHERWISE)
-ARISING IN ANY WAY OUT OF THE USE OF THIS SOFTWARE, EVEN IF ADVISED OF THE POSSIBILITY OF SUCH DAMAGE.
+THIS SOFTWARE IS PROVIDED BY THE COPYRIGHT HOLDERS AND CONTRIBUTORS "AS IS" AND ANY EXPRESS OR
+IMPLIED WAR-
+RANTIES, INCLUDING, BUT NOT LIMITED TO, THE IMPLIED WARRANTIES OF MERCHANTABILITY AND FITNESS FOR A
+PARTICULAR
+PURPOSE ARE DISCLAIMED. IN NO EVENT SHALL THE COPYRIGHT HOLDER OR CONTRIBUTORS BE LIABLE FOR ANY
+DIRECT, IN-
+DIRECT, INCIDENTAL, SPECIAL, EXEMPLARY, OR CONSEQUENTIAL DAMAGES (INCLUDING, BUT NOT LIMITED TO,
+PROCUREMENT
+OF SUBSTITUTE GOODS OR SERVICES; LOSS OF USE, DATA, OR PROFITS; OR BUSINESS INTERRUPTION) HOWEVER
+CAUSED AND
+ON ANY THEORY OF LIABILITY, WHETHER IN CONTRACT, STRICT LIABILITY, OR TORT (INCLUDING NEGLIGENCE OR
+OTHERWISE)
+ARISING IN ANY WAY OUT OF THE USE OF THIS SOFTWARE, EVEN IF ADVISED OF THE POSSIBILITY OF SUCH
+DAMAGE.
 -->
 <robot name="husky" xmlns:xacro="http://ros.org/wiki/xacro">
@@ -38,20 +49,21 @@
   <xacro:arg name="robot_namespace" default="/husky" />
   <xacro:arg name="urdf_extras" default="empty.urdf" />
-  <xacro:arg name="transmission_hw_interface" default="false"/>
+  <xacro:arg name="transmission_hw_interface" default="false" />
   <!-- Included URDF/XACRO Files -->
   <xacro:include filename="$(find husky_ur3_gazebo)/urdf/decorations.urdf.xacro" />
   <xacro:include filename="$(find husky_ur3_gazebo)/urdf/wheel.urdf.xacro" />
-  <xacro:include filename="$(find husky_ur3_gazebo)/urdf/accessories/sensor_arch.urdf.xacro"/>
-  <xacro:include filename="$(find husky_ur3_gazebo)/urdf/accessories/sick_tim571.urdf.xacro"/>
+  <xacro:include filename="$(find husky_ur3_gazebo)/urdf/accessories/sensor_arch.urdf.xacro" />
+  <xacro:include filename="$(find husky_ur3_gazebo)/urdf/accessories/sick_tim571.urdf.xacro" />
   <xacro:if value="$(arg transmission_hw_interface)">
-    <xacro:include filename="$(find husky_ur3_gazebo)/urdf/ur3_robot_gripper_effort.urdf.xacro"/>
+    <xacro:include filename="$(find husky_ur3_gazebo)/urdf/ur3_robot_gripper_effort.urdf.xacro" />
   </xacro:if>
   <xacro:unless value="$(arg transmission_hw_interface)">
-    <xacro:include filename="$(find husky_ur3_gazebo)/urdf/ur3_robot_gripper.urdf.xacro"/>
+    <xacro:include filename="$(find husky_ur3_gazebo)/urdf/ur3_robot_gripper.urdf.xacro" />
   </xacro:unless>
-  <xacro:include filename="$(find husky_ur3_gazebo)/urdf/accessories/d435_camera_h.urdf.xacro"/>
-  <xacro:include filename="$(find husky_ur3_gazebo)/urdf/accessories/d435_camera_g.urdf.xacro"/>
-  <!--xacro:include filename="$(find husky_ur3_gazebo)/urdf/ur3_robot.urdf.xacro"/-->
-  <xacro:property name="M_PI" value="3.14159"/>
+  <xacro:include filename="$(find husky_ur3_gazebo)/urdf/accessories/d435_camera_h.urdf.xacro" />
+  <xacro:include filename="$(find husky_ur3_gazebo)/urdf/accessories/d435_camera_g.urdf.xacro" />
+  <!--xacro:include
+  filename="$(find husky_ur3_gazebo)/urdf/ur3_robot.urdf.xacro"/-->
+  <xacro:property name="M_PI" value="3.14159" />
   <!-- Base Size -->
   <xacro:property name="base_x_size" value="0.98740000" />
@@ -73,19 +85,22 @@
       </geometry>
     </visual>
-    <collision>
-      <origin xyz="${( husky_front_bumper_extend - husky_rear_bumper_extend ) / 2.0} 0 ${base_z_size/4}" rpy="0 0 0" />
-      <geometry>
-        <box size="${ base_x_size + husky_front_bumper_extend + husky_rear_bumper_extend } ${base_y_size} ${base_z_size/2}"/>
+    <collision name="base_collision1">
+      <origin
+        xyz="${( husky_front_bumper_extend - husky_rear_bumper_extend ) / 2.0} 0 ${base_z_size/4}"
+        rpy="0 0 0" />
+      <geometry>
+        <box
+          size="${ base_x_size + husky_front_bumper_extend + husky_rear_bumper_extend } ${base_y_size + 0.12} ${base_z_size/2}" />
       </geometry>
     </collision>
-    <collision>
+    <collision name="base_collision2">
       <origin xyz="0 0 ${base_z_size*3/4-0.01}" rpy="0 0 0" />
       <geometry>
-        <box size="${base_x_size*4/5} ${base_y_size} ${base_z_size/2-0.02}"/>
+        <box size="${base_x_size*4/5} ${base_y_size + 0.12} ${base_z_size/2-0.02}" />
       </geometry>
     </collision>
   </link>
   <!-- Base footprint is on the ground under the robot -->
-  <link name="base_footprint"/>
+  <link name="base_footprint" />
   <joint name="base_footprint_joint" type="fixed">
     <origin xyz="0 0 ${wheel_vertical_offset - wheel_radius}" rpy="0 0 0" />
@@ -108,7 +123,8 @@
   <!-- IMU Link is the standard mounting position for the UM6 IMU.-->
   <!-- Can be modified with environment variables in /etc/ros/setup.bash -->
-  <link name="imu_link"/>
+  <link name="imu_link" />
   <joint name="imu_joint" type="fixed">
-    <origin xyz="$(optenv HUSKY_IMU_XYZ 0.19 0 0.149)" rpy="$(optenv HUSKY_IMU_RPY 0 -1.5708 3.1416)" />
+    <origin xyz="$(optenv HUSKY_IMU_XYZ 0.19 0 0.149)"
+      rpy="$(optenv HUSKY_IMU_RPY 0 -1.5708 3.1416)" />
     <parent link="base_link" />
     <child link="imu_link" />
@@ -130,44 +146,44 @@
   </xacro:husky_wheel>
   <gazebo reference="front_left_wheel_link">
-		  <material>Gazebo/DarkGrey</material>
-      <selfCollide>false</selfCollide>
-      <mu1 value="1.0"/>
-      <mu2 value="1.0"/>
-      <kp value="10000000.0" />
-      <kd value="1" />
-      <fdir1 value="1 0 0"/>
-	</gazebo>
-	<gazebo reference="rear_left_wheel_link">
-		 <material>Gazebo/DarkGrey</material>
-      <selfCollide>false</selfCollide>
-      <mu1 value="0.05"/>
-      <mu2 value="0.05"/>
-      <kp value="10000000.0" />
-      <kd value="1" />
-      <fdir1 value="1 0 0"/>
-	</gazebo>
-    <gazebo reference="front_right_wheel_link">
-		  <material>Gazebo/DarkGrey</material>
-      <selfCollide>false</selfCollide>
-      <mu1 value="1.0"/>
-      <mu2 value="1.0"/>
-      <kp value="10000000.0" />
-      <kd value="1" />
-      <fdir1 value="1 0 0"/>
-	</gazebo>
-	<gazebo reference="rear_right_wheel_link">
-		<material>Gazebo/DarkGrey</material>
-      <selfCollide>false</selfCollide>
-      <mu1 value="0.05"/>
-      <mu2 value="0.05"/>
-      <kp value="10000000.0" />
-      <kd value="1" />
-      <fdir1 value="1 0 0"/>
-	</gazebo>
+    <material>Gazebo/DarkGrey</material>
+    <selfCollide>false</selfCollide>
+    <mu1 value="1.0" />
+    <mu2 value="1.0" />
+    <kp value="10000000.0" />
+    <kd value="1" />
+    <fdir1 value="1 0 0" />
+  </gazebo>
+  <gazebo reference="rear_left_wheel_link">
+    <material>Gazebo/DarkGrey</material>
+    <selfCollide>false</selfCollide>
+    <mu1 value="0.05" />
+    <mu2 value="0.05" />
+    <kp value="10000000.0" />
+    <kd value="1" />
+    <fdir1 value="1 0 0" />
+  </gazebo>
+  <gazebo reference="front_right_wheel_link">
+    <material>Gazebo/DarkGrey</material>
+    <selfCollide>false</selfCollide>
+    <mu1 value="1.0" />
+    <mu2 value="1.0" />
+    <kp value="10000000.0" />
+    <kd value="1" />
+    <fdir1 value="1 0 0" />
+  </gazebo>
+  <gazebo reference="rear_right_wheel_link">
+    <material>Gazebo/DarkGrey</material>
+    <selfCollide>false</selfCollide>
+    <mu1 value="0.05" />
+    <mu2 value="0.05" />
+    <kp value="10000000.0" />
+    <kd value="1" />
+    <fdir1 value="1 0 0" />
+  </gazebo>
   <xacro:husky_decorate />
   <xacro:sensor_sick_tim571 prefix="front_laser" parent="top_plate_link" prefix_topic="front_laser">
-   	<origin xyz="$(arg laser_xyz)" rpy="$(arg laser_rpy)"/>
+    <origin xyz="$(arg laser_xyz)" rpy="$(arg laser_rpy)" />
   </xacro:sensor_sick_tim571>
-<!--  <xacro:if value="$(arg camera_h_enabled)">
+  <!--  <xacro:if value="$(arg camera_h_enabled)">
     <xacro:h_sensor_d435 parent="top_plate_link">
       <origin xyz="$(arg camera_h_xyz)" rpy="$(arg camera_h_rpy)"/>
@@ -180,29 +196,30 @@
   </xacro:if>
 -->
- <joint name="control_box_ur3_joint" type="fixed">
-      <origin xyz="-0.095 0 0.233" rpy="${M_PI/2} 0 0" />
-      <parent link="top_plate_link"/>
-      <child link="control_box_ur3_link" />
-    </joint>
+  <joint name="control_box_ur3_joint" type="fixed">
+    <origin xyz="-0.095 0 0.233" rpy="${M_PI/2} 0 0" />
+    <parent link="top_plate_link" />
+    <child link="control_box_ur3_link" />
+  </joint>
   <link name="control_box_ur3_link">
     <inertial>
       <mass value="5.0" />
       <origin xyz="0 0 0" />
-      <inertia  ixx="0.0" ixy="0.0"  ixz="0.0"  iyy="0.0"  iyz="0.0"  izz="0.0" />
+      <inertia ixx="0.0" ixy="0.0" ixz="0.0" iyy="0.0" iyz="0.0" izz="0.0" />
     </inertial>
     <visual>
-       <origin xyz="0 0 0" rpy="0 -${M_PI/2} 0 " />
-       <geometry>
-         <mesh filename="package://husky_ur3_gazebo/meshes/UR_Contorl_Box.stl" scale="0.001 0.001 0.001"/>
-       </geometry>
-       <material name="gray">
-         <color rgba="0.153 0.153 0.153 1"/>
-       </material>
+      <origin xyz="0 0 0" rpy="0 -${M_PI/2} 0 " />
+      <geometry>
+        <mesh filename="package://husky_ur3_gazebo/meshes/UR_Contorl_Box.stl"
+          scale="0.001 0.001 0.001" />
+      </geometry>
+      <material name="gray">
+        <color rgba="0.153 0.153 0.153 1" />
+      </material>
     </visual>
     <collision>
-       <origin xyz="-0.1 0 0" rpy="0 0 0 " />
-       <geometry>
-           <box size="0.28 0.46 0.37"/>
-       </geometry>
+      <origin xyz="-0.1 0 0" rpy="0 0 0 " />
+      <geometry>
+        <box size="0.28 0.46 0.37" />
+      </geometry>
     </collision>
   </link>
@@ -248,18 +265,78 @@
   <gazebo>
     <plugin name="gazebo_grasp_fix" filename="libgazebo_grasp_fix.so">
-        <arm>
-          <arm_name>ur3_robot</arm_name>
-          <palm_link> wrist_3_link  </palm_link>
-          <gripper_link> rh_p12_rn_r2 </gripper_link>
-          <gripper_link> rh_p12_rn_l2 </gripper_link>
-        </arm>
-        <forces_angle_tolerance>100</forces_angle_tolerance>
-        <update_rate>4</update_rate>
-        <grip_count_threshold>4</grip_count_threshold>
-        <max_grip_count>8</max_grip_count>
-        <release_tolerance>0.005</release_tolerance>
-        <disable_collisions_on_attach>false</disable_collisions_on_attach>
-        <contact_topic>__default_topic__</contact_topic>
-    </plugin>
+      <arm>
+        <arm_name>ur3_robot</arm_name>
+        <palm_link> wrist_3_link </palm_link>
+        <gripper_link> rh_p12_rn_r2 </gripper_link>
+        <gripper_link> rh_p12_rn_l2 </gripper_link>
+      </arm>
+      <forces_angle_tolerance>100</forces_angle_tolerance>
+      <update_rate>4</update_rate>
+      <grip_count_threshold>4</grip_count_threshold>
+      <max_grip_count>8</max_grip_count>
+      <release_tolerance>0.005</release_tolerance>
+      <disable_collisions_on_attach>false</disable_collisions_on_attach>
+      <contact_topic>__default_topic__</contact_topic>
+    </plugin>
+  </gazebo>
+  <gazebo>
+    <plugin name="p3d_base_controller" filename="libgazebo_ros_p3d.so">
+      <alwaysOn>true</alwaysOn>
+      <updateRate>50.0</updateRate>
+      <bodyName>base_footprint</bodyName>
+      <topicName>base_pose_ground_truth</topicName>
+      <gaussianNoise>0.01</gaussianNoise>
+      <frameName>map</frameName>
+      <xyzOffsets>0 0 0</xyzOffsets>
+      <rpyOffsets>0 0 0</rpyOffsets>
+    </plugin>
+  </gazebo>
+  <gazebo reference="base_link">
+    <!-- Virtual Contact Sensor -->
+    <sensor name='base_contact_sensor' type='contact'>
+      <contact>
+        <collision>base_link_fixed_joint_lump__base_collision1_collision</collision>
+      </contact>
+      <plugin name="my_plugin" filename="libgazebo_ros_bumper.so">
+        <bumperTopicName>base_collision_0</bumperTopicName>
+        <frameName>base_link</frameName>
+      </plugin>
+    </sensor>
+  </gazebo>
+  <gazebo reference="base_link">
+    <!-- Virtual Contact Sensor -->
+    <sensor name='base_contact_sensor2' type='contact'>
+      <contact>
+        <collision>base_link_fixed_joint_lump__base_collision2_collision_1</collision>
+      </contact>
+      <plugin name="my_plugin2" filename="libgazebo_ros_bumper.so">
+        <bumperTopicName>base_collision_1</bumperTopicName>
+        <frameName>base_link</frameName>
+      </plugin>
+    </sensor>
+  </gazebo>
+  <gazebo reference="rear_bumper_link">
+    <!-- Virtual Contact Sensor -->
+    <sensor name='base_contact_sensor3' type='contact'>
+      <contact>
+        <collision>base_link_fixed_joint_lump__rear_bumper_collision_collision_3</collision>
+      </contact>
+      <plugin name="my_plugin3" filename="libgazebo_ros_bumper.so">
+        <bumperTopicName>base_collision_2</bumperTopicName>
+        <frameName>base_link</frameName>
+      </plugin>
+    </sensor>
+  </gazebo>
+  <gazebo reference="front_bumper_link">
+    <!-- Virtual Contact Sensor -->
+    <sensor name='base_contact_sensor4' type='contact'>
+      <contact>
+        <collision>base_link_fixed_joint_lump__front_bumper_collision_collision_2</collision>
+      </contact>
+      <plugin name="my_plugin4" filename="libgazebo_ros_bumper.so">
+        <bumperTopicName>base_collision_3</bumperTopicName>
+        <frameName>base_link</frameName>
+      </plugin>
+    </sensor>
   </gazebo>
 </robot>
